Commit message: completed uw ros control

File: src/urdf/uw.urdf (robot description, URDF)
Before this commit: robot uhugv, 9 links, 8 joints
Links:
- link base_link: mass 0.79826 -> 1.0
- link servoL_mount_1: mass 0.79826 -> 0.2
- link servoL_mount_2: mass 0.79826 -> 0.2
- link servoL_mount_3: mass 0.79826 -> 0.2
- link servoL_mount_4: mass 0.79826 -> 0.2
- link servoR_mount_1: mass 0.79826 -> 0.2
- link servoR_mount_2: mass 0.79826 -> 0.2
- link servoR_mount_3: mass 0.79826 -> 0.2
- link servoR_mount_4: mass 0.79826 -> 0.2
Joints:
- joint servoL_1: origin xyz=0 0 0 rpy=0 0 0 -> xyz=0.21 0.31 0.14 rpy=0 0 0
- joint servoL_2: origin xyz=0 0 0 rpy=0 0 0 -> xyz=0.11 0.31 0.14 rpy=0 0 0
- joint servoL_3: origin xyz=0 0 0 rpy=0 0 0 -> xyz=0.0 0.31 0.14 rpy=0 0 0
- joint servoL_4: origin xyz=0 0 0 rpy=0 0 0 -> xyz=-0.11 0.31 0.14 rpy=0 0 0
- joint servoR_1: origin xyz=0 0 0 rpy=0 0 0 -> xyz=0.21 -0.31 0.14 rpy=0 0 0
- joint servoR_2: origin xyz=0 0 0 rpy=0 0 0 -> xyz=0.11 -0.31 0.14 rpy=0 0 0
- joint servoR_3: origin xyz=0 0 0 rpy=0 0 0 -> xyz=0.0 -0.31 0.14 rpy=0 0 0
- joint servoR_4: origin xyz=0 0 0 rpy=0 0 0 -> xyz=-0.11 -0.31 0.14 rpy=0 0 0

Commit message: added uw publisher

File: src/urdf/uw.urdf (robot description, URDF)
Before this commit: robot track, 9 links, 8 joints
Links:
- link base_link: geometry collision box size=0.548 0.656 0.182; visual mesh filename=package://uhugv/meshes/uhugv.dae
- link servoL_mount_1: geometry collision box size=0.1 0.2 0.01; visual mesh filename=package://uhugv/meshes/servo.dae
- link servoL_mount_2: geometry collision box size=0.1 0.2 0.01; visual mesh filename=package://uhugv/meshes/servo.dae
- link servoL_mount_3: geometry collision box size=0.1 0.2 0.01; visual mesh filename=package://uhugv/meshes/servo.dae
- link servoL_mount_4: geometry collision box size=0.1 0.2 0.01; visual mesh filename=package://uhugv/meshes/servo.dae
- link servoR_mount_1: geometry collision box size=0.1 0.2 0.01; visual mesh filename=package://uhugv/meshes/servo.dae
- link servoR_mount_2: geometry collision box size=0.1 0.2 0.01; visual mesh filename=package://uhugv/meshes/servo.dae
- link servoR_mount_3: geometry collision box size=0.1 0.2 0.01; visual mesh filename=package://uhugv/meshes/servo.dae
- link servoR_mount_4: geometry collision box size=0.1 0.2 0.01; visual mesh filename=package://uhugv/meshes/servo.dae

Commit message: update readme.md

File: src/urdf/uw.urdf (robot description, URDF)
Before this commit: robot track, 9 links, 8 joints
Links:
- link servoL_mount_1: geometry collision box size=0.1 0.02 0.01; visual mesh filename=package://uhugv/meshes/servo.dae
- link servoL_mount_2: geometry collision box size=0.1 0.02 0.01; visual mesh filename=package://uhugv/meshes/servo.dae
- link servoL_mount_3: geometry collision box size=0.1 0.02 0.01; visual mesh filename=package://uhugv/meshes/servo.dae
- link servoL_mount_4: geometry collision box size=0.1 0.02 0.01; visual mesh filename=package://uhugv/meshes/servo.dae
- link servoR_mount_1: geometry collision box size=0.1 0.02 0.01; visual mesh filename=package://uhugv/meshes/servo.dae
- link servoR_mount_2: geometry collision box size=0.1 0.02 0.01; visual mesh filename=package://uhugv/meshes/servo.dae
- link servoR_mount_3: geometry collision box size=0.1 0.02 0.01; visual mesh filename=package://uhugv/meshes/servo.dae
- link servoR_mount_4: geometry collision box size=0.1 0.02 0.01; visual mesh filename=package://uhugv/meshes/servo.dae
